Commit message: Gazebo simulation and update README

File: src/swd_starter_kit_description/urdf/swd_starter_kit.urdf (robot description, URDF)
Before this commit: robot swd_starter_kit, 8 links, 7 joints
Links:
- link base_link: geometry collision mesh filename=file:///home/fatma/autonomous_slam_baseline/src/swd_starter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 scale=0.001 0.001 0.001; visual box size=0.55 0.40 0.01
- link swd_left_link: geometry collision cylinder length=0.037 radius=0.0630; visual mesh filename=file:///home/fatma/autonomous_slam_baseline/src/swd_starter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 scale=0.001 0.001 0.001
- link swd_right_link: geometry collision cylinder length=0.037 radius=0.0630; visual mesh filename=file:///home/fatma/autonomous_slam_baseline/src/swd_starter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 scale=0.001 0.001 0.001
